File: Boards/LPM_AJ_BEDOFNAILS/Bed_of_nails/Bed_of_nails.kicad_sch (KiCad schematic)
At the start: 62 parts, among them J1 TU, J10 TU1, J11 TU2, J12 TU3, J13 TU4, J2 TD, J3 V+RS485, J4 PT, J5 Conn_ZIF_9, J6 TD1, J7 TD2, J8 TD3, J9 TD4, U1 Conn_ZIF_5pos

Commit message: added relay
Still needs better separation between the AC lines and footprints relay need fixing
Parts:
- J1, J2, J3: Farnell (none) -> 2827902
- J4: Farnell (none) -> 1593490
- J5: Farnell (none) -> 3215773
- TP1, TP10, TP11, TP12, TP13, TP14, TP15, TP16, TP17, TP18, TP19, TP2, TP20, TP21, TP22, TP23, TP24, TP25, TP26, TP27, TP28, TP29, TP3, TP30, TP31, TP32, TP33, TP34, TP35, TP36, TP37, TP38, TP39, TP4, TP40, TP41, TP42, TP43, TP44, TP45, TP46, TP47, TP48, TP5, TP6, TP7, TP8, TP9: footprint MyFootprints:KS-075-47-G-10_KS-07547G10 -> MyFootPrints:INGUN_KS-075-47-G-10_KS-07547G10
- U1: Farnell (none) -> 3215771
