File: Boards/TestBoardArduino/Connectors.kicad_sch (KiCad schematic)
At the start: 39 parts, among them J1 TU, J2 TD, J3 PT, J4 V+RS485, J5 UART, K2 MCHRS1KH-S DC24V, K3 MCHRS1KH-S DC24V, Q4 DMN6068SE-13, Q5 DMN6068SE-13

Commit message: Updated board
Parts:
- added C8: 220uF, Capacitor_SMD:CP_Elec_10x10, symbol Device:C_Polarized_Small
- R33: value 320R -> 5k1
Connections:
- net +5VP is gone; now on net +24V: D10.1 (K), J5.1 (Pin_1), R33.1
- net +24V: now also C8.1
- net GND: now also C8.2
Changed lines of the file:
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@@
 	)
 	(junction
+		(at 182.88 27.178)
+		(diameter 0)
+		(color 0 0 0 0)
+	)
+	(junction
+		(at 175.514 27.178)
+		(diameter 0)
+		(color 0 0 0 0)
+	)
+	(junction
 		(at 64.897 114.046)
 		(diameter 0)
@@
 	)
 	(junction
+		(at 162.052 27.178)
+		(diameter 0)
+		(color 0 0 0 0)
+	)
+	(junction
 		(at 22.987 140.716)
 		(diameter 0)
@@
 	)
 	(junction
-		(at 182.88 27.432)
-		(diameter 0)
-		(color 0 0 0 0)
-	)
-	(junction
 		(at 173.99 87.122)
 		(diameter 0)
@@
 	)
 	(junction
-		(at 204.47 27.432)
-		(diameter 0)
-		(color 0 0 0 0)
-	)
-	(junction
 		(at 64.897 116.586)
 		(diameter 0)
@@
 	(wire
 		(pts
+			(xy 182.88 27.178) (xy 182.88 31.75)
+		)
+		(stroke
+			(width 0)
+			(type default)
+		)
+	)
+	(wire
+		(pts
 			(xy 64.897 111.506) (xy 64.897 114.046)
 		)
@@
 	(wire
 		(pts
+			(xy 162.052 40.386) (xy 162.052 43.434)
+		)
+		(stroke
+			(width 0)
+			(type default)
+		)
+	)
+	(wire
+		(pts
 			(xy 152.146 80.01) (xy 152.146 81.788)
 		)
@@
 	(wire
 		(pts
+			(xy 162.052 27.178) (xy 162.052 35.306)
+		)
+		(stroke
+			(width 0)
+			(type default)
+		)
+	)
+	(wire
+		(pts
 			(xy 204.216 41.402) (xy 204.216 46.482)
 		)
@@
 	(wire
 		(pts
-			(xy 182.88 27.432) (xy 204.47 27.432)
+			(xy 182.88 27.178) (xy 204.47 27.178)
+		)
+		(stroke
+			(width 0)
+			(type default)
+		)
+	)
+	(wire
+		(pts
+			(xy 175.514 27.178) (xy 162.052 27.178)
 		)
 		(stroke
@@
 	(wire
 		(pts
-			(xy 175.514 27.432) (xy 175.514 35.052)
+			(xy 175.514 27.178) (xy 175.514 35.052)
 		)
 		(stroke
@@
 	(wire
 		(pts
-			(xy 175.514 27.432) (xy 182.88 27.432)
+			(xy 175.514 27.178) (xy 182.88 27.178)
 		)
 		(stroke
@@
 	(wire
 		(pts
-			(xy 50.292 103.886) (xy 64.897 103.886)
+			(xy 162.052 26.162) (xy 162.052 27.178)
 		)
 		(stroke
@@
 	(wire
 		(pts
-			(xy 22.987 145.796) (xy 37.592 145.796)
-		)
-		(stroke
-			(width 0)
-			(type default)
-		)
-	)
-	(wire
-		(pts
-			(xy 22.987 103.886) (xy 22.987 106.426)
+			(xy 50.292 103.886) (xy 64.897 103.886)
 		)
 		(stroke
@@
 	(wire
 		(pts
-			(xy 60.452 76.454) (xy 64.008 76.454)
+			(xy 22.987 145.796) (xy 37.592 145.796)
 		)
 		(stroke
@@
 	(wire
 		(pts
-			(xy 234.95 114.808) (xy 234.95 116.078)
+			(xy 22.987 103.886) (xy 22.987 106.426)
 		)
 		(stroke
@@
 	(wire
 		(pts
-			(xy 204.47 33.782) (xy 204.47 27.432)
+			(xy 60.452 76.454) (xy 64.008 76.454)
 		)
 		(stroke
@@
 	(wire
 		(pts
-			(xy 159.512 84.328) (xy 180.34 84.328)
+			(xy 234.95 114.808) (xy 234.95 116.078)
 		)
 		(stroke
@@
 	(wire
 		(pts
-			(xy 204.47 27.432) (xy 204.47 22.86)
+			(xy 204.47 27.178) (xy 204.47 33.782)
 		)
 		(stroke
@@
 	(wire
 		(pts
-			(xy 182.88 27.432) (xy 182.88 31.75)
+			(xy 159.512 84.328) (xy 180.34 84.328)
 		)
 		(stroke
@@
 	(symbol
 		(lib_id "power:GND")
+		(at 162.052 43.434 0)
+		(unit 1)
+		(exclude_from_sim no)
+		(in_bom yes)
+		(on_board yes)
+		(dnp no)
+		(fields_autoplaced yes)
+		(property "Reference" "#PWR033"
+			(at 162.052 49.784 0)
+			(effects
+				(font
+					(size 1.27 1.27)
+				)
+				(hide yes)
+			)
+		)
+		(property "Value" "GND"
+			(at 162.052 48.514 0)
+			(effects
+				(font
+					(size 1.27 1.27)
+				)
+			)
+		)
+		(property "Footprint" ""
+			(at 162.052 43.434 0)
+			(effects
+				(font
+					(size 1.27 1.27)
+				)
+				(hide yes)
+			)
+		)
+		(property "Datasheet" ""
+			(at 162.052 43.434 0)
+			(effects
+				(font
+					(size 1.27 1.27)
+				)
+				(hide yes)
+			)
+		)
+		(property "Description" ""
+			(at 162.052 43.434 0)
+			(effects
+				(font
+					(size 1.27 1.27)
+				)
+				(hide yes)
+			)
+		)
+		(pin "1"
+		)
+		(instances
+			(project "TestBoardArduino"
+				(path "/569848bc-480b-4cfe-96a1-7f07584b7f26/cf6ded4f-36cd-4b46-bf8f-208e0333a6e4"
+					(reference "#PWR033")
+					(unit 1)
+				)
+			)
+		)
+	)
+	(symbol
+		(lib_id "power:GND")
 		(at 61.722 180.721 0)
 		(unit 1)
@@
 		(fields_autoplaced yes)
 		(property "Reference" "R33"
-			(at 185.42 33.02 0)
+			(at 185.42 33.0199 0)
 			(effects
 				(font
@@
 			)
 		)
-		(property "Value" "320R"
-			(at 185.42 35.56 0)
+		(property "Value" "5k1"
+			(at 185.42 35.5599 0)
 			(effects
 				(font
@@
 	)
 	(symbol
+		(lib_name "+24V_1")
+		(lib_id "power:+24V")
+		(at 162.052 26.162 0)
+		(unit 1)
+		(exclude_from_sim no)
+		(in_bom yes)
+		(on_board yes)
+		(dnp no)
+		(fields_autoplaced yes)
+		(property "Reference" "#PWR029"
+			(at 162.052 29.972 0)
+			(effects
+				(font
+					(size 1.27 1.27)
+				)
+				(hide yes)
+			)
+		)
+		(property "Value" "+24V"
+			(at 162.052 21.844 0)
+			(effects
+				(font
+					(size 1.27 1.27)
+				)
+			)
+		)
+		(property "Footprint" ""
+			(at 162.052 26.162 0)
+			(effects
+				(font
+					(size 1.27 1.27)
+				)
+				(hide yes)
+			)
+		)
+		(property "Datasheet" ""
+			(at 162.052 26.162 0)
+			(effects
+				(font
+					(size 1.27 1.27)
+				)
+				(hide yes)
+			)
+		)
+		(property "Description" "Power symbol creates a global label with name \"+24V\""
+			(at 162.052 26.162 0)
+			(effects
+				(font
+					(size 1.27 1.27)
+				)
+				(hide yes)
+			)
+		)
+		(pin "1"
+		)
+		(instances
+			(project "TestBoardArduino"
+				(path "/569848bc-480b-4cfe-96a1-7f07584b7f26/cf6ded4f-36cd-4b46-bf8f-208e0333a6e4"
+					(reference "#PWR029")
+					(unit 1)
+				)
+			)
+		)
+	)
+	(symbol
 		(lib_id "Device:R")
 		(at 180.34 100.965 0)
@@
 	)
 	(symbol
-		(lib_id "power:+5VP")
-		(at 204.47 22.86 0)
+		(lib_id "Device:C_Polarized_Small")
+		(at 162.052 37.846 0)
 		(unit 1)
 		(exclude_from_sim no)
@@
 		(dnp no)
 		(fields_autoplaced yes)
-		(property "Reference" "#PWR033"
-			(at 204.47 26.67 0)
+		(property "Reference" "C8"
+			(at 165.227 36.0298 0)
 			(effects
 				(font
 					(size 1.27 1.27)
 				)
-				(hide yes)
+				(justify left)
 			)
 		)
-		(property "Value" "+5VP"
-			(at 204.47 17.78 0)
+		(property "Value" "220uF"
+			(at 165.227 38.5698 0)
 			(effects
 				(font
 					(size 1.27 1.27)
 				)
+				(justify left)
 			)
 		)
-		(property "Footprint" ""
-			(at 204.47 22.86 0)
+		(property "Footprint" "Capacitor_SMD:CP_Elec_10x10"
+			(at 162.052 37.846 0)
 			(effects
 				(font
@@
 			)
 		)
-		(property "Datasheet" ""
-			(at 204.47 22.86 0)
+		(property "Datasheet" "~"
+			(at 162.052 37.846 0)
+			(effects
+				(font
+					(size 1.27 1.27)
+				)
+				(hide yes)
+			)
+		)
+		(property "Description" ""
+			(at 162.052 37.846 0)
 			(effects
 				(font
@@
 			)
 		)
-		(property "Description" "Power symbol creates a global label with name \"+5VP\""
-			(at 204.47 22.86 0)
+		(property "Farnell" "2471976"
+			(at 162.052 37.846 0)
 			(effects
 				(font
@@
 		(pin "1"
 		)
+		(pin "2"
+		)
 		(instances
 			(project "TestBoardArduino"
 				(path "/569848bc-480b-4cfe-96a1-7f07584b7f26/cf6ded4f-36cd-4b46-bf8f-208e0333a6e4"
-					(reference "#PWR033")
+					(reference "C8")
 					(unit 1)
 				)
