File: Boards/TestBoardArduino/PS.kicad_sch (KiCad schematic)
At the start: 22 parts, among them J8 2007986, U10 XC6902N331MR-G, U6 LM2937IMP-5.0/NOPB, U7 LM2940IMP-12/NOPB, U8 MAX889TESA+

Commit message: Updated board
Parts:
- removed C8: 220uF, Capacitor_SMD:CP_Elec_10x10, symbol Device:C_Polarized_Small
- removed F1: 1A, Fuse:Fuse_0402_1005Metric_Pad0.77x0.64mm_HandSolder, symbol Device:Fuse
- removed FB1: MMZ2012Y600BT000, Capacitor_SMD:C_0805_2012Metric_Pad1.18x1.45mm_HandSolder, symbol Device:FerriteBead_Small
- removed J8: 2007986, MyFootPrints:Screwterminal_3mm81_3pos, symbol Connector:Screw_Terminal_01x03
- removed PS1: IRM-15-24, MyFootPrints:IRM-15-24, symbol Converter_ACDC:IRM-02-15
